Commit message: 能跑起来了

File: carsim_discription/urdf/model.urdf (robot description, URDF)
Before this commit: robot basic_car, 8 links, 7 joints
Links:
- removed link hokuyo_link

Commit message: 把模型改回原来的了

File: carsim_discription/urdf/model.urdf (robot description, URDF)
Before this commit: robot basic_car, 7 links, 7 joints
Links:
- added link hokuyo_link, mass 1e-5; collision box size=0.1 0.1 0.1; visual mesh filename=package://carsim_discription/meshes/hokuyo.dae
